File: EXTERNAL_LED_BOARD/EXTERNAL_LED_BOARD.kicad_pcb (KiCad board)
At the start: 2 copper layers, 27 x 17 mm, 8 parts, among them J1 Conn_01x05_Male, J2 Conn_01x05_Male, U1 WS2812-2020

Commit message: update
Parts:
- removed U1: WS2812-2020, footprint:LED_WS2812-2020
- added C2: C_Small, Capacitor_SMD:C_0603_1608Metric_Pad1.05x0.95mm_HandSolder, F.Cu at (136.9, 99.0)
- added C3: C_Small, Capacitor_SMD:C_0603_1608Metric_Pad1.05x0.95mm_HandSolder, F.Cu at (132.5, 99.0)
- added LED1: WS2812C-2020, SamacSys_Parts:WS2812C2020, F.Cu at (139.1, 99.0)
- added LED2: WS2812C-2020, SamacSys_Parts:WS2812C2020, F.Cu at (134.7, 99.0)
- added LED3: WS2812C-2020, SamacSys_Parts:WS2812C2020, F.Cu at (130.3, 99.0)
- J1, J2: value Conn_01x05_Male -> B03B-PASK-1__LF___SN_; footprint footprint:B05B-PASK-1 -> SamacSys_Parts:B03BPASK1LFSN
- moved J1 11.5 mm to (134.7, 93.4), turned to 0 degrees
- moved J2 11.4 mm to (134.7, 104.7)
- moved C1 2.71 mm to (141.3, 99.0)
Connections:
- J1 pad 3: /OUT -> GND
- J1 pad 4: Net-(J1-Pad4) -> (no net)
- J2 pad 2: /IN -> /OUT
- J2 pad 3: /OUT -> GND
- J2 pad 4: Net-(J2-Pad4) -> (no net)
Routing:
- net /OUT: track 23.9 -> 6.68 mm
- net /IN: track 21.0 -> 5.87 mm
- net Net-(LED1-Pad3): track 0.00 -> 14.1 mm, vias 0 -> 2
- net Net-(LED2-Pad3): track 0.00 -> 14.1 mm, vias 0 -> 2
- net +5V: track 30.4 -> 32.1 mm
- net GND: track 12.4 -> 13.5 mm
Other:
- board text added: "5V"
- board text added: "GND"
- board text added: "IN"
- board text added: "OUT"
