File: EXTERNAL_LED_BOARD/EXTERNAL_LED_BOARD.sch (KiCad schematic (older format))
At the start: 8 parts, among them J1 Conn_01x05_Male, J2 Conn_01x05_Male, U1 WS2812-2020

Commit message: update
Parts:
- removed J1, J2: Conn_01x05_Male, footprint:B05B-PASK-1, symbol Connector:Conn_01x05_Male
- removed U1: WS2812-2020, footprint:LED_WS2812-2020, symbol WS2812-2020:WS2812-2020
- added C2, C3: C_Small, Capacitor_SMD:C_0603_1608Metric_Pad1.05x0.95mm_HandSolder, symbol Device:C_Small
- added J1, J2: B03B-PASK-1__LF___SN_, SamacSys_Parts:B03BPASK1LFSN, symbol SamacSys_Parts:B03B-PASK-1__LF___SN_
- added LED1, LED2, LED3: WS2812C-2020, SamacSys_Parts:WS2812C2020, symbol SamacSys_Parts:WS2812C-2020
Connections:
- net +5V: now also C2.1, C3.1, J1.1, J2.1, LED1.4 (VDD), LED2.4 (VDD), LED3.4 (VDD)
- net GND: now also C2.2, C3.2, J1.3, J2.3, LED1.2 (GND), LED2.2 (GND), LED3.2 (GND)
- net IN: now also J1.2, LED3.3 (DI)
- net OUT: now also J2.2, LED1.1 (DO)
- new net: LED2.3 (DI), LED3.1 (DO)
- new net: LED1.3 (DI), LED2.1 (DO)
- no-connect marks 2 -> 0
